File: arduino/pcb/aop/aop.kicad_pcb (KiCad board)
At the start: 2 copper layers, 0 parts

Commit message: PCB: start tracing
Parts:
- added BZ1: Buzzer, Buzzer_Beeper:Buzzer_12x9.5RM7.6, F.Cu at (74.9, 126.0)
- added D1: LED, LED_THT:LED_D3.0mm, B.Cu at (92.7, 80.0)
- added J1: Conn_01x02_Pin, Connector_JST:JST_XH_B2B-XH-A_1x02_P2.50mm_Vertical, F.Cu at (75.5, 90.0)
- added M1: RFID-RC522, RFID-RC522:RFID-RC522, B.Cu at (92.0, 117.5)
- added Q1: AO4435, AO4435:SOIC127P600X175-8N, F.Cu at (89.5, 90.1)
- added R1: 100K, Resistor_THT:R_Axial_DIN0207_L6.3mm_D2.5mm_P10.16mm_Horizontal, F.Cu at (101.0, 98.2)
- added R2: 1K, Resistor_THT:R_Axial_DIN0207_L6.3mm_D2.5mm_P10.16mm_Horizontal, F.Cu at (105.0, 98.2)
- added R3: 100, Resistor_THT:R_Axial_DIN0207_L6.3mm_D2.5mm_P10.16mm_Horizontal, F.Cu at (109.0, 98.2)
- added SW1: SW_Push, Resistor_THT:R_Axial_DIN0614_L14.3mm_D5.7mm_P20.32mm_Horizontal, F.Cu at (108.5, 125.5)
- added U1: ESP32-C3_SUPERMINI_TH, ESP32-C3_SUPERMINI_TH:MODULE_ESP32-C3_SUPERMINI_TH, F.Cu at (85.4, 105.6)
- added U2: TC00500, TC00500:MODULE_TC00500, F.Cu at (73.5, 73.8)
Routing:
- net GND: track 0.00 -> 71.7 mm
- net Net-(U1-GPIO21): track 0.00 -> 34.4 mm
- net Net-(Q1-Pad4): track 0.00 -> 29.7 mm
- net Net-(U1-3V3): track 0.00 -> 29.1 mm
- net Net-(M1-SDA): track 0.00 -> 23.3 mm
- net Net-(M1-MOSI): track 0.00 -> 20.5 mm
- net Net-(M1-MISO): track 0.00 -> 20.2 mm
- net Net-(U1-GPIO0): track 0.00 -> 18.2 mm
- net Net-(D1-A): track 0.00 -> 17.0 mm
- net +BATT: track 0.00 -> 8.00 mm
